Commit message: Update robot.urdf

File: urdf/robot.urdf (robot description, URDF)
Before this commit: robot visual, 13 links, 12 joints
Joints:
- joint left_back_wheel_joint: type prismatic -> fixed
- joint left_front_wheel_joint: type prismatic -> fixed
- joint right_back_wheel_joint: type continuous -> fixed
- joint right_front_wheel_joint: type continuous -> fixed
